File: KiCad/GR_Wifi_Current_Trigger.kicad_pcb (KiCad board)
At the start: 2 copper layers, 43.7 x 27.9 mm, 14 parts, among them J1 3.5mm Jack, J2 Conn_01x03, U1 LM358, U2 WeMos_D1_mini

Commit message: Add files via upload
Parts:
- added C5: 47uF, Capacitor_THT:CP_Radial_D5.0mm_P2.50mm, F.Cu at (122.2, 90.6)
- moved R1 3.90 mm to (136.1, 90.9)
- moved R2 3.80 mm to (125.9, 88.0)
- moved C2 1.30 mm to (118.2, 90.9)
Routing:
- net Net-(C2-Pad1): track 14.6 -> 19.7 mm
- net /Triggered: track 47.7 -> 45.4 mm
- net +5V: track 47.8 -> 49.6 mm

Commit message: Add files via upload
Parts:
- C5: value 47uF -> DNI
- R1: value 10K -> 47K
- R2: value 4K7 -> 47K
Connections:
- R1 pad 1: +5V -> +3V3
- U2 pad 8: Net-(U2-Pad8) -> +3V3
Routing:
- net +5V: track 49.6 -> 27.3 mm, vias 2 -> 0
- net +3V3: track 0.00 -> 11.8 mm
